Commit message: 修改urdf,j2和j3向上2度,旧版本存储在piper_description_old中

File: src/piper_description/urdf/piper_no_gripper_description_old.urdf (robot description, URDF)
Before this commit: robot piper, 10 links, 9 joints
Links:
- removed link gripper_base
- removed link link7
- removed link link8
Joints:
- removed joint joint6_to_gripper_base
- removed joint joint7
- removed joint joint8
- joint joint2: origin xyz=0 0 0 rpy=1.5708 -0.1359 -3.1416 -> xyz=0 0 0 rpy=1.5708 -0.10095 -3.1416
- joint joint3: origin xyz=0.28503 0 0 rpy=0 0 -1.7939 -> xyz=0.28503 0 0 rpy=0 0 -1.759
