Commit message: 增加匹诺曹机械臂逆解

File: src/piper_description/urdf/piper_description.urdf (robot description, URDF)
Before this commit: robot piper_description, 9 links, 8 joints
Links:
- link link6: geometry collision mesh filename=package://piper_description/meshes/link6_1.STL; visual mesh filename=package://piper_description/meshes/link6.dae
Joints:
- joint joint6: origin xyz=0 0.091 0.0014165 rpy=-1.5708 -1.5708 0 -> xyz=0 0.091 0.0014165 rpy=-1.5708 -3.1415926 0
- joint joint7: origin xyz=0 0 0.13503 rpy=1.5708 0 1.5708 -> xyz=0 0 0.13503 rpy=1.5708 0 3.1415926
- joint joint8: origin xyz=0 0 0.13503 rpy=-1.5708 0 1.5708 -> xyz=0 0 0.13503 rpy=-1.5708 0 3.1415926

File: src/piper_description/urdf/piper_description.xacro (robot description, xacro)
@@ -359,5 +359,5 @@
       <origin
         xyz="0 0 0"
-        rpy="0 0 0" />
+        rpy="0 0 1.5708" />
       <geometry>
         <mesh
@@ -376,5 +376,5 @@
       <geometry>
         <mesh
-          filename="package://piper_description/meshes/link6.STL" />
+          filename="package://piper_description/meshes/link6_1.STL" />
       </geometry>
     </collision>
@@ -385,5 +385,5 @@
     <origin
       xyz="0 0.091 0.0014165"
-      rpy="-1.5708 -1.5708 0" />
+      rpy="-1.5708 -3.1415926 0" />
     <parent
       link="link5" />
@@ -443,5 +443,5 @@
     <origin
       xyz="0 0 0.13503"
-      rpy="1.5708 0 1.5708" />
+      rpy="1.5708 0 3.1415926" />
     <parent
       link="link6" />
@@ -501,5 +501,5 @@
     <origin
       xyz="0 0 0.13503"
-      rpy="-1.5708 0 1.5708" />
+      rpy="-1.5708 0 3.1415926" />
     <parent
       link="link6" />

Commit message: 更新urdf

File: src/piper_description/urdf/piper_description.urdf (robot description, URDF)
Before this commit: robot piper_description, 9 links, 8 joints
Links:
- added link gripper_base, mass 0.145318531013916; collision mesh filename=package://piper_description/meshes/gripper_base.STL; visual mesh filename=package://piper_description/meshes/gripper_base.STL
- link base_link: mass 0.162548567403693 -> 0.333893486740112; geometry collision mesh filename=package://piper_description/meshes/base_link.STL; visual mesh filename=package://piper_description/meshes/base_link.STL
- link link1: mass 0.0978679932242825 -> 0.215052383265765; geometry collision mesh filename=package://piper_description/meshes/link1.STL; visual mesh filename=package://piper_description/meshes/link1.STL
- link link2: mass 0.290888938633388 -> 0.463914239236335; geometry collision mesh filename=package://piper_description/meshes/link2.STL; visual mesh filename=package://piper_description/meshes/link2.STL
- link link3: mass 0.290847697793211 -> 0.219942452993132; geometry collision mesh filename=package://piper_description/meshes/link3.STL; visual mesh filename=package://piper_description/meshes/link3.STL
- link link4: mass 0.127087348341362 -> 0.131814339939458; geometry collision mesh filename=package://piper_description/meshes/link4.STL; visual mesh filename=package://piper_description/meshes/link4.STL
- link link5: mass 0.144711242639457 -> 0.134101341225523; geometry collision mesh filename=package://piper_description/meshes/link5.STL; visual mesh filename=package://piper_description/meshes/link5.STL
- link link6: mass 0.195187143240719 -> 0.00699089613564366; geometry collision mesh filename=package://piper_description/meshes/link6.STL; visual mesh filename=package://piper_description/meshes/link6.STL
- link link7: mass 0.02648229234527 -> 0.0303534920715906; geometry collision mesh filename=package://piper_description/meshes/link7.STL; visual mesh filename=package://piper_description/meshes/link7.STL
- link link8: mass 0.0264822021416248 -> 0.0303534920715904; geometry collision mesh filename=package://piper_description/meshes/link8.STL; visual mesh filename=package://piper_description/meshes/link8.STL
Joints:
- added joint joint6_to_gripper_base: type fixed, parent link6, child gripper_base, origin xyz=0 0 0 rpy=0 0 0
- joint joint1: limit lower=-2.618 upper=2.618 effort=100 velocity=3 -> lower=-2.618 upper=2.168 effort=100 velocity=5; origin xyz=0 0 0.123 rpy=0 0 -1.5708 -> xyz=0 0 0.123 rpy=0 0 0
- joint joint2: limit lower=0 upper=3.14 effort=100 velocity=3 -> lower=0 upper=3.14 effort=100 velocity=5; origin xyz=0 0 0 rpy=1.5708 0 -1.5708 -> xyz=0 0 0 rpy=1.5708 -0.10095 -3.1416
- joint joint3: limit lower=-2.697 upper=0 effort=100 velocity=3 -> lower=-2.697 upper=0 effort=100 velocity=5; origin xyz=0.28358 0.028726 0 rpy=0 0 0.10095 -> xyz=0.28503 0 0 rpy=0 0 -1.759
- joint joint4: limit lower=-1.832 upper=1.832 effort=100 velocity=3 -> lower=-1.832 upper=1.832 effort=100 velocity=5; origin xyz=-0.24221 0.068514 0 rpy=-1.5708 0 1.3826 -> xyz=-0.021984 -0.25075 0 rpy=1.5708 0 0
- joint joint5: limit lower=-1.22 upper=1.22 effort=100 velocity=3 -> lower=-1.22 upper=1.22 effort=100 velocity=5; origin xyz=0 0 0 rpy=1.5708 0 0 -> xyz=0 0 0 rpy=-1.5708 0 0
- joint joint6: limit lower=-3.14 upper=3.14 effort=100 velocity=3 -> lower=-2.0944 upper=2.0944 effort=100 velocity=3; origin xyz=0 0.091 0.0014165 rpy=-1.5708 -3.1415926 0 -> xyz=8.8259E-05 -0.091 0 rpy=1.5708 0 0
- joint joint7: axis 0 0 -1 -> 0 0 1; limit lower=0 upper=0.04 effort=10 velocity=1 -> lower=0 upper=0.035 effort=10 velocity=1; origin xyz=0 0 0.13503 rpy=1.5708 0 3.1415926 -> xyz=0 0 0.1358 rpy=1.5708 0 0; parent link6 -> gripper_base
- joint joint8: axis 0 0 1 -> 0 0 -1; limit lower=-0.04 upper=0 effort=10 velocity=1 -> lower=-0.035 upper=0 effort=10 velocity=1; origin xyz=0 0 0.13503 rpy=-1.5708 0 3.1415926 -> xyz=0 0 0.1358 rpy=1.5708 0 -3.1416; parent link6 -> gripper_base

File: src/piper_description/urdf/piper_description.xacro (robot description, xacro)
@@ -14,31 +14,17 @@
     <inertial>
       <origin
-        xyz="-0.00979274765955341 1.82905827587138E-06 0.0410100126360189"
-        rpy="0 0 0" />
-      <mass
-        value="0.162548567403693" />
-      <inertia
-        ixx="0.000226596924525071"
-        ixy="-7.33972270153965E-08"
-        ixz="2.13249977802622E-06"
-        iyy="0.000269444772561524"
-        iyz="8.15169009611054E-09"
-        izz="0.000222318258878636" />
-    </inertial>
-    <visual>
-      <origin
-        xyz="0 0 0"
-        rpy="0 0 0" />
-      <geometry>
-        <mesh
-          filename="package://piper_description/meshes/base_link.dae" />
-      </geometry>
-      <material
-        name="">
-        <color
-          rgba="0.792156862745098 0.819607843137255 0.933333333333333 1" />
-      </material>
-    </visual>
-    <collision>
+        xyz="-0.00473641164191482 2.56829134630247E-05 0.041451518036016"
+        rpy="0 0 0" />
+      <mass
+        value="0.333893486740112" />
+      <inertia
+        ixx="0.000254953479570424"
+        ixy="2.06931238580746E-07"
+        ixz="7.30912474718368E-06"
+        iyy="0.00027202099920186"
+        iyz="2.65131745382267E-07"
+        izz="0.000276534627629623" />
+    </inertial>
+    <visual>
       <origin
         xyz="0 0 0"
@@ -48,4 +34,18 @@
           filename="package://piper_description/meshes/base_link.STL" />
       </geometry>
+      <material
+        name="">
+        <color
+          rgba="0.792156862745098 0.819607843137255 0.933333333333333 1" />
+      </material>
+    </visual>
+    <collision>
+      <origin
+        xyz="0 0 0"
+        rpy="0 0 0" />
+      <geometry>
+        <mesh
+          filename="package://piper_description/meshes/base_link.STL" />
+      </geometry>
     </collision>
   </link>
@@ -54,23 +54,23 @@
     <inertial>
       <origin
-        xyz="0.00131676031927024 0.000310288842008612 -0.00922874512303437"
-        rpy="0 0 0" />
-      <mass
-        value="0.0978679932242825" />
-      <inertia
-        ixx="7.76684558296782E-05"
-        ixy="1.09084650459924E-07"
-        ixz="-1.9748053243241E-06"
-        iyy="9.24967780161547E-05"
-        iyz="9.91284646834582E-07"
-        izz="8.24589062407807E-05" />
-    </inertial>
-    <visual>
-      <origin
-        xyz="0 0 0"
-        rpy="0 0 0" />
-      <geometry>
-        <mesh
-          filename="package://piper_description/meshes/link1.dae" />
+        xyz="0.000121504734057468 0.000104632162460536 -0.00438597309559853"
+        rpy="0 0 0" />
+      <mass
+        value="0.215052383265765" />
+      <inertia
+        ixx="0.000109639007860341"
+        ixy="2.50631260865109E-07"
+        ixz="-1.89352789149844E-07"
+        iyy="9.95612262461418E-05"
+        iyz="1.00634716976093E-08"
+        izz="0.000116363910317385" />
+    </inertial>
+    <visual>
+      <origin
+        xyz="0 0 0"
+        rpy="0 0 0" />
+      <geometry>
+        <mesh
+          filename="package://piper_description/meshes/link1.STL" />
       </geometry>
       <material
@@ -95,5 +95,5 @@
     <origin
       xyz="0 0 0.123"
-      rpy="0 0 -1.5708" />
+      rpy="0 0 0" />
     <parent
       link="base_link" />
@@ -104,7 +104,7 @@
     <limit
       lower="-2.618"
-      upper="2.618"
+      upper="2.168"
       effort="100"
-      velocity="3" />
+      velocity="5" />
   </joint>
   <link
@@ -112,23 +112,23 @@
     <inertial>
       <origin
-        xyz="0.148793602378802 -0.00242026983944119 0.00175154638467948"
-        rpy="0 0 0" />
-      <mass
-        value="0.290888938633388" />
-      <inertia
-        ixx="0.000148959640166183"
-        ixy="-7.37750384371657E-05"
-        ixz="-9.68688405196236E-07"
-        iyy="0.00172800946632652"
-        iyz="-1.09692225564224E-06"
-        izz="0.0017754628344594" />
-    </inertial>
-    <visual>
-      <origin
-        xyz="0 0 0"
-        rpy="0 0 0" />
-      <geometry>
-        <mesh
-          filename="package://piper_description/meshes/link2.dae" />
+        xyz="0.198666145229743 -0.010926924140076 0.00142121714502687"
+        rpy="0 0 0" />
+      <mass
+        value="0.463914239236335" />
+      <inertia
+        ixx="0.000214137415059993"
+        ixy="7.26120579340088E-05"
+        ixz="-9.88224861011274E-07"
+        iyy="0.00100030277518254"
+        iyz="-1.32818212212246E-06"
+        izz="0.00104417184176783" />
+    </inertial>
+    <visual>
+      <origin
+        xyz="0 0 0"
+        rpy="0 0 0" />
+      <geometry>
+        <mesh
+          filename="package://piper_description/meshes/link2.STL" />
       </geometry>
       <material
@@ -153,5 +153,5 @@
     <origin
       xyz="0 0 0"
-      rpy="1.5708 0 -1.5708" />
+      rpy="1.5708 -0.10095 -3.1416" />
     <parent
       link="link1" />
@@ -164,5 +164,5 @@
       upper="3.14"
       effort="100"
-      velocity="3" />
+      velocity="5" />
   </joint>
   <link
@@ -170,23 +170,23 @@
     <inertial>
       <origin
-        xyz="-0.0996835215213704 0.0349477226691318 0.000508025815507312"
-        rpy="0 0 0" />
-      <mass
-        value="0.290847697793211" />
-      <inertia
-        ixx="0.000107879011637167"
-        ixy="2.92669521203626E-05"
-        ixz="6.825922326238E-07"
-        iyy="0.000214751671792086"
-        iyz="-7.78469047878196E-07"
-        izz="0.000241923439340319" />
-    </inertial>
-    <visual>
-      <origin
-        xyz="0 0 0"
-        rpy="0 0 0" />
-      <geometry>
-        <mesh
-          filename="package://piper_description/meshes/link3.dae" />
+        xyz="-0.0202737662122021 -0.133914995944595 -0.000458682652737356"
+        rpy="0 0 0" />
+      <mass
+        value="0.219942452993132" />
+      <inertia
+        ixx="0.00018953849076141"
+        ixy="-8.05719205057736E-06"
+        ixz="5.10255053956334E-07"
+        iyy="7.1424497082494E-05"
+        iyz="8.89044974368937E-07"
+        izz="0.000201212938725775" />
+    </inertial>
+    <visual>
+      <origin
+        xyz="0 0 0"
+        rpy="0 0 0" />
+      <geometry>
+        <mesh
+          filename="package://piper_description/meshes/link3.STL" />
       </geometry>
       <material
@@ -210,6 +210,6 @@
     type="revolute">
     <origin
-      xyz="0.28358 0.028726 0"
-      rpy="0 0 0.10095" />
+      xyz="0.28503 0 0"
+      rpy="0 0 -1.759" />
     <parent
       link="link2" />
@@ -222,5 +222,5 @@
       upper="0"
       effort="100"
-      velocity="3" />
+      velocity="5" />
   </joint>
   <link
@@ -228,23 +228,23 @@
     <inertial>
       <origin
-        xyz="0.000276464622387979 -0.00102803669324875 -0.00472830700561663"
-        rpy="0 0 0" />
-      <mass
-        value="0.127087348341362" />
-      <inertia
-        ixx="3.82011730423416E-05"
-        ixy="-4.92358350897513E-08"
-        ixz="4.89589432973119E-08"
-        iyy="4.87048555222578E-05"
-        iyz="6.70802942500512E-08"
-        izz="4.10592077565559E-05" />
-    </inertial>
-    <visual>
-      <origin
-        xyz="0 0 0"
-        rpy="0 0 0" />
-      <geometry>
-        <mesh
-          filename="package://piper_description/meshes/link4.dae" />
+        xyz="-9.66635791618542E-05 0.000876064475651083 -0.00496880904640868"
+        rpy="0 0 0" />
+      <mass
+        value="0.131814339939458" />
+      <inertia
+        ixx="3.96965423235175E-05"
+        ixy="-2.32268338444837E-08"
+        ixz="-1.14702090783249E-07"
+        iyy="5.13319789853892E-05"
+        iyz="9.92852686264567E-08"
+        izz="4.14768131680711E-05" />
+    </inertial>
+    <visual>
+      <origin
+        xyz="0 0 0"
+        rpy="0 0 0" />
+      <geometry>
+        <mesh
+          filename="package://piper_description/meshes/link4.STL" />
       </geometry>
       <material
@@ -268,6 +268,6 @@
     type="revolute">
     <origin
-      xyz="-0.24221 0.068514 0"
-      rpy="-1.5708 0 1.3826" />
+      xyz="-0.021984 -0.25075 0"
+      rpy="1.5708 0 0" />
     <parent
       link="link3" />
@@ -280,5 +280,5 @@
       upper="1.832"
       effort="100"
-      velocity="3" />
+      velocity="5" />
   </joint>
   <link
@@ -286,23 +286,23 @@
     <inertial>
       <origin
-        xyz="8.82262433516967E-05 0.0566829014808256 -0.00196119720482461"
-        rpy="0 0 0" />
-      <mass
-        value="0.144711242639457" />
-      <inertia
-        ixx="4.39644313662493E-05"
-        ixy="-3.59259686444846E-08"
-        ixz="-1.89747741386183E-08"
-        iyy="5.63173920951307E-05"
-        iyz="-2.1540716689785E-07"
-        izz="4.88713664675268E-05" />
-    </inertial>
-    <visual>
-      <origin
-        xyz="0 0 0"
-        rpy="0 0 0" />
-      <geometry>
-        <mesh
-          filename="package://piper_description/meshes/link5.dae" />
+        xyz="-4.10554118924211E-05 -0.0566486692356075 -0.0037205791677906"
+        rpy="0 0 0" />
+      <mass
+        value="0.134101341225523" />
+      <inertia
+        ixx="4.10994130543451E-05"
+        ixy="-2.06433983793957E-08"
+        ixz="1.29591347668502E-10"
+        iyy="5.27723004189144E-05"
+        iyz="1.9140716904272E-07"
+        izz="4.60418752810541E-05" />
+    </inertial>
+    <visual>
+      <origin
+        xyz="0 0 0"
+        rpy="0 0 0" />
+      <geometry>
+        <mesh
+          filename="package://piper_description/meshes/link5.STL" />
       </geometry>
       <material
@@ -327,5 +327,5 @@
     <origin
       xyz="0 0 0"
-      rpy="1.5708 0 0" />
+      rpy="-1.5708 0 0" />
     <parent
       link="link4" />
@@ -338,5 +338,5 @@
       upper="1.22"
       effort="100"
-      velocity="3" />
+      velocity="5" />
   </joint>
   <link
@@ -344,37 +344,37 @@
     <inertial>
       <origin
-        xyz="0.00103120214523473 0.0121761387587524 0.0315480874960164"
-        rpy="0 0 0" />
-      <mass
-        value="0.195187143240719" />
-      <inertia
-        ixx="6.43790256535539E-05"
-        ixy="-1.2366166157046E-06"
-        ixz="1.97664606328472E-07"
-        iyy="0.000126146396374301"
-        iyz="2.41157078516408E-06"
-        izz="0.000154087076816444" />
-    </inertial>
-    <visual>
-      <origin
-        xyz="0 0 0"
-        rpy="0 0 1.5708" />
-      <geometry>
-        <mesh
-          filename="package://piper_description/meshes/link6.dae" />
-      </geometry>
-      <material
-        name="">
-        <color
-          rgba="0.792156862745098 0.819607843137255 0.933333333333333 1" />
-      </material>
-    </visual>
-    <collision>
-      <origin
-        xyz="0 0 0"
-        rpy="0 0 0" />
-      <geometry>
-        <mesh
-          filename="package://piper_description/meshes/link6_1.STL" />
+        xyz="-8.82590762930069E-05 9.0598378529832E-06 -0.002"
+        rpy="0 0 0" />
+      <mass
+        value="0.00699089613564366" />
+      <inertia
+        ixx="5.43015540542155E-07"
+        ixy="-1.98305403089247E-22"
+        ixz="-7.2791893904596E-23"
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
File: src/piper_description/urdf/piper_no_gripper_description.urdf (robot description, URDF)
Before this commit: robot piper_description, 6 links, 5 joints
Links:
- added link link6, mass 0.00699089613564366; collision mesh filename=package://piper_description/meshes/link6.STL; visual mesh filename=package://piper_description/meshes/link6.STL
- link base_link: mass 0.162548567403693 -> 0.333893486740112; geometry collision mesh filename=package://piper_description/meshes/base_link.STL; visual mesh filename=package://piper_description/meshes/base_link.STL
- link link1: mass 0.0978679932242825 -> 0.215052383265765; geometry collision mesh filename=package://piper_description/meshes/link1.STL; visual mesh filename=package://piper_description/meshes/link1.STL
- link link2: mass 0.290888938633388 -> 0.463914239236335; geometry collision mesh filename=package://piper_description/meshes/link2.STL; visual mesh filename=package://piper_description/meshes/link2.STL
- link link3: mass 0.290847697793211 -> 0.219942452993132; geometry collision mesh filename=package://piper_description/meshes/link3.STL; visual mesh filename=package://piper_description/meshes/link3.STL
- link link4: mass 0.127087348341362 -> 0.131814339939458; geometry collision mesh filename=package://piper_description/meshes/link4.STL; visual mesh filename=package://piper_description/meshes/link4.STL
- link link5: mass 0.144711242639457 -> 0.134101341225523; geometry collision mesh filename=package://piper_description/meshes/link5.STL; visual mesh filename=package://piper_description/meshes/link5.STL
Joints:
- added joint joint6: type revolute, parent link5, child link6, origin xyz=8.8259E-05 -0.091 0 rpy=1.5708 0 0, axis 0 0 1, limit lower=-2.0944 upper=2.0944 effort=100 velocity=5
- joint joint1: limit lower=-2.618 upper=2.618 effort=100 velocity=3 -> lower=-2.618 upper=2.168 effort=100 velocity=5; origin xyz=0 0 0.123 rpy=0 0 -1.5708 -> xyz=0 0 0.123 rpy=0 0 0
- joint joint2: limit lower=0 upper=3.14 effort=100 velocity=3 -> lower=0 upper=3.14 effort=100 velocity=5; origin xyz=0 0 0 rpy=1.5708 0 -1.5708 -> xyz=0 0 0 rpy=1.5708 -0.10095 -3.1416
- joint joint3: limit lower=-2.697 upper=0 effort=100 velocity=3 -> lower=-2.697 upper=0 effort=100 velocity=5; origin xyz=0.28358 0.028726 0 rpy=0 0 0.10095 -> xyz=0.28503 0 0 rpy=0 0 -1.759
- joint joint4: limit lower=-1.832 upper=1.832 effort=100 velocity=3 -> lower=-1.832 upper=1.832 effort=100 velocity=5; origin xyz=-0.24221 0.068514 0 rpy=-1.5708 0 1.3826 -> xyz=-0.021984 -0.25075 0 rpy=1.5708 0 0
- joint joint5: limit lower=-1.22 upper=1.22 effort=100 velocity=3 -> lower=-1.22 upper=1.22 effort=100 velocity=5; origin xyz=0 0 0 rpy=1.5708 0 0 -> xyz=0 0 0 rpy=-1.5708 0 0
