Commit message: 整合piper_ros_moveit和piper_sim到piper_ros,修正urdf的质量和惯性矩阵,统一piper_description

File: src/piper_description/urdf/piper_description.urdf (robot description, URDF)
Before this commit: robot piper_description, 10 links, 9 joints
Links:
- link base_link: mass 0.333893486740112 -> 1.02
- link gripper_base: mass 0.145318531013916 -> 0.45
- link link1: mass 0.215052383265765 -> 0.71
- link link2: mass 0.463914239236335 -> 1.17
- link link3: mass 0.219942452993132 -> 0.5
- link link4: mass 0.131814339939458 -> 0.38
- link link5: mass 0.134101341225523 -> 0.383
- link link7: mass 0.0303534920715906 -> 0.025
- link link8: mass 0.0303534920715904 -> 0.025

File: src/piper_description/urdf/piper_description.xacro (robot description, xacro)
@@ -1,5 +1,5 @@
 <?xml version="1.0" encoding="utf-8"?>
 <robot
-  name="arm"
+  name="piper"
   xmlns:xacro="http://ros.org/wiki/xacro">
 <!-- world -->
@@ -9,5 +9,5 @@
       <child link="base_link"/>
   </joint>
-<!-- arm -->
+<!-- piper -->
 <link
     name="base_link">
@@ -17,12 +17,12 @@
         rpy="0 0 0" />
       <mass
-        value="0.333893486740112" />
-      <inertia
-        ixx="0.000254953479570424"
-        ixy="2.06931238580746E-07"
-        ixz="7.30912474718368E-06"
-        iyy="0.00027202099920186"
-        iyz="2.65131745382267E-07"
-        izz="0.000276534627629623" />
+        value="1.02" />
+      <inertia
+        ixx="0.00267433"
+        ixy="-0.00000073"
+        ixz="-0.00017389"
+        iyy="0.00282612"
+        iyz="0.0000004"
+        izz="0.00089624" />
     </inertial>
     <visual>
@@ -57,12 +57,12 @@
         rpy="0 0 0" />
       <mass
-        value="0.215052383265765" />
-      <inertia
-        ixx="0.000109639007860341"
-        ixy="2.50631260865109E-07"
-        ixz="-1.89352789149844E-07"
-        iyy="9.95612262461418E-05"
-        iyz="1.00634716976093E-08"
-        izz="0.000116363910317385" />
+        value="0.71" />
+      <inertia
+        ixx="0.00048916"
+        ixy="-0.00000036"
+        ixz="-0.00000224"
+        iyy="0.00040472"
+        iyz="-0.00000242"
+        izz="0.00043982" />
     </inertial>
     <visual>
@@ -115,12 +115,12 @@
         rpy="0 0 0" />
       <mass
-        value="0.463914239236335" />
-      <inertia
-        ixx="0.000214137415059993"
-        ixy="7.26120579340088E-05"
-        ixz="-9.88224861011274E-07"
-        iyy="0.00100030277518254"
-        iyz="-1.32818212212246E-06"
-        izz="0.00104417184176783" />
+        value="1.17" />
+      <inertia
+        ixx="0.00116918"
+        ixy="-0.00180037"
+        ixz="0.00025146"
+        iyy="0.06785384"
+        iyz="-0.00000455"
+        izz="0.06774489" />
     </inertial>
     <visual>
@@ -173,12 +173,12 @@
         rpy="0 0 0" />
       <mass
-        value="0.219942452993132" />
-      <inertia
-        ixx="0.00018953849076141"
-        ixy="-8.05719205057736E-06"
-        ixz="5.10255053956334E-07"
-        iyy="7.1424497082494E-05"
-        iyz="8.89044974368937E-07"
-        izz="0.000201212938725775" />
+        value="0.5" />
+      <inertia
+        ixx="0.01361711"
+        ixy="0.00165794"
+        ixz="-0.00000048"
+        iyy="0.00045024"
+        iyz="-0.00000045"
+        izz="0.01380322" />
     </inertial>
     <visual>
@@ -231,12 +231,12 @@
         rpy="0 0 0" />
       <mass
-        value="0.131814339939458" />
-      <inertia
-        ixx="3.96965423235175E-05"
-        ixy="-2.32268338444837E-08"
-        ixz="-1.14702090783249E-07"
-        iyy="5.13319789853892E-05"
-        iyz="9.92852686264567E-08"
-        izz="4.14768131680711E-05" />
+        value="0.38" />
+      <inertia
+        ixx="0.00018501"
+        ixy="0.00000054"
+        ixz="0.00000120"
+        iyy="0.00018965"
+        iyz="-0.00000841"
+        izz="0.00015484" />
     </inertial>
     <visual>
@@ -289,12 +289,12 @@
         rpy="0 0 0" />
       <mass
-        value="0.134101341225523" />
-      <inertia
-        ixx="4.10994130543451E-05"
-        ixy="-2.06433983793957E-08"
-        ixz="1.29591347668502E-10"
-        iyy="5.27723004189144E-05"
-        iyz="1.9140716904272E-07"
-        izz="4.60418752810541E-05" />
+        value="0.383" />
+      <inertia
+        ixx="0.00166169"
+        ixy="0.00000006"
+        ixz="-0.00000007"
+        iyy="0.00018510"
+        iyz="0.00001026"
+        izz="0.00164321" />
     </inertial>
     <visual>
@@ -349,8 +349,8 @@
         value="0.00699089613564366" />
       <inertia
-        ixx="5.43015540542155E-07"
+        ixx="5.73015540542155E-07"
         ixy="-1.98305403089247E-22"
         ixz="-7.2791893904596E-23"
-        iyy="5.43015540542155E-07"
+        iyy="5.73015540542155E-07"
         iyz="-3.4146026640245E-24"
         izz="1.06738869138926E-06" />
@@ -405,12 +405,12 @@
         rpy="0 0 0" />
       <mass
-        value="0.145318531013916" />
-      <inertia
-        ixx="0.000101740348396288"
-        ixy="-1.43961090652723E-07"
-        ixz="-8.72352812740139E-08"
-        iyy="4.16518088621566E-05"
-        iyz="3.27712901952435E-08"
-        izz="0.000118691325723675" />
+        value="0.45" />
+      <inertia
+        ixx="0.00092934"
+        ixy="0.00000034"
+        ixz="-0.00000738"
+        iyy="0.00071447"
+        iyz="0.00000005"
+        izz="0.00039442" />
     </inertial>
     <visual>
@@ -456,12 +456,12 @@
         rpy="0 0 0" />
       <mass
-        value="0.0303534920715906" />
-      <inertia
-        ixx="1.13870358991284E-05"
-        ixy="4.2853410993302E-07"
-        ixz="-6.45170690459141E-08"
-        iyy="6.26108891787743E-06"
-        iyz="1.5729036212893E-06"
-        izz="1.57822030592869E-05" />
+        value="0.025" />
+      <inertia
+        ixx="0.00007371"
+        ixy="-0.00000113"
+        ixz="0.00000021"
+        iyy="0.00000781"
+        iyz="-0.00001372"
+        izz="0.0000747" />
     </inertial>
     <visual>
@@ -514,12 +514,12 @@
         rpy="0 0 0" />
       <mass
-        value="0.0303534920715904" />
-      <inertia
-        ixx="1.13870358991283E-05"
-        ixy="4.28534109932964E-07"
-        ixz="-6.45170690459078E-08"
-        iyy="6.26108891787742E-06"
-        iyz="1.57290362128933E-06"
-        izz="1.57822030592867E-05" />
+        value="0.025" />
+      <inertia
+        ixx="0.00007371"
+        ixy="-0.00000113"
+        ixz="0.00000021"
+        iyy="0.00000781"
+        iyz="-0.00001372"
+        izz="0.0000747" />
     </inertial>
     <visual>
@@ -589,5 +589,5 @@
   <gazebo>
     <plugin name="gazebo_ros_control" filename="libgazebo_ros_control.so">
-        <robotNamespace>/piper_description</robotNamespace>
+        <robotNamespace>/piper</robotNamespace>
         <legacyModeNS>true</legacyModeNS>
     </plugin>

File: src/piper_description/urdf/piper_no_gripper_description.urdf (robot description, URDF)
Before this commit: robot piper_description, 7 links, 6 joints
Links:
- link base_link: mass 0.333893486740112 -> 1.02
- link link1: mass 0.215052383265765 -> 0.71
- link link2: mass 0.463914239236335 -> 1.17
- link link3: mass 0.219942452993132 -> 0.5
- link link4: mass 0.131814339939458 -> 0.38
- link link5: mass 0.134101341225523 -> 0.383
Joints:
- joint joint6: limit lower=-2.0944 upper=2.0944 effort=100 velocity=5 -> lower=-2.0944 upper=2.0944 effort=100 velocity=3

File: src/piper_description/urdf/piper_no_gripper_description.xacro (robot description, xacro)
@@ -1,5 +1,5 @@
 <?xml version="1.0" encoding="utf-8"?>
 <robot
-  name="arm"
+  name="piper"
   xmlns:xacro="http://ros.org/wiki/xacro">
 <!-- world -->
@@ -9,5 +9,5 @@
       <child link="base_link"/>
   </joint>
-<!-- arm -->
+<!-- piper -->
 <link
     name="base_link">
@@ -17,12 +17,12 @@
         rpy="0 0 0" />
       <mass
-        value="0.333893486740112" />
-      <inertia
-        ixx="0.000254953479570424"
-        ixy="2.06931238580746E-07"
-        ixz="7.30912474718368E-06"
-        iyy="0.00027202099920186"
-        iyz="2.65131745382267E-07"
-        izz="0.000276534627629623" />
+        value="1.02" />
+      <inertia
+        ixx="0.00267433"
+        ixy="-0.00000073"
+        ixz="-0.00017389"
+        iyy="0.00282612"
+        iyz="0.0000004"
+        izz="0.00089624" />
     </inertial>
     <visual>
@@ -57,12 +57,12 @@
         rpy="0 0 0" />
       <mass
-        value="0.215052383265765" />
-      <inertia
-        ixx="0.000109639007860341"
-        ixy="2.50631260865109E-07"
-        ixz="-1.89352789149844E-07"
-        iyy="9.95612262461418E-05"
-        iyz="1.00634716976093E-08"
-        izz="0.000116363910317385" />
+        value="0.71" />
+      <inertia
+        ixx="0.00048916"
+        ixy="-0.00000036"
+        ixz="-0.00000224"
+        iyy="0.00040472"
+        iyz="-0.00000242"
+        izz="0.00043982" />
     </inertial>
     <visual>
@@ -115,12 +115,12 @@
         rpy="0 0 0" />
       <mass
-        value="0.463914239236335" />
-      <inertia
-        ixx="0.000214137415059993"
-        ixy="7.26120579340088E-05"
-        ixz="-9.88224861011274E-07"
-        iyy="0.00100030277518254"
-        iyz="-1.32818212212246E-06"
-        izz="0.00104417184176783" />
+        value="1.17" />
+      <inertia
+        ixx="0.00116918"
+        ixy="-0.00180037"
+        ixz="0.00025146"
+        iyy="0.06785384"
+        iyz="-0.00000455"
+        izz="0.06774489" />
     </inertial>
     <visual>
@@ -173,12 +173,12 @@
         rpy="0 0 0" />
       <mass
-        value="0.219942452993132" />
-      <inertia
-        ixx="0.00018953849076141"
-        ixy="-8.05719205057736E-06"
-        ixz="5.10255053956334E-07"
-        iyy="7.1424497082494E-05"
-        iyz="8.89044974368937E-07"
-        izz="0.000201212938725775" />
+        value="0.5" />
+      <inertia
+        ixx="0.01361711"
+        ixy="0.00165794"
+        ixz="-0.00000048"
+        iyy="0.00045024"
+        iyz="-0.00000045"
+        izz="0.01380322" />
     </inertial>
     <visual>
@@ -231,12 +231,12 @@
         rpy="0 0 0" />
       <mass
-        value="0.131814339939458" />
-      <inertia
-        ixx="3.96965423235175E-05"
-        ixy="-2.32268338444837E-08"
-        ixz="-1.14702090783249E-07"
-        iyy="5.13319789853892E-05"
-        iyz="9.92852686264567E-08"
-        izz="4.14768131680711E-05" />
+        value="0.38" />
+      <inertia
+        ixx="0.00018501"
+        ixy="0.00000054"
+        ixz="0.00000120"
+        iyy="0.00018965"
+        iyz="-0.00000841"
+        izz="0.00015484" />
     </inertial>
     <visual>
@@ -289,12 +289,12 @@
         rpy="0 0 0" />
       <mass
-        value="0.134101341225523" />
-      <inertia
-        ixx="4.10994130543451E-05"
-        ixy="-2.06433983793957E-08"
-        ixz="1.29591347668502E-10"
-        iyy="5.27723004189144E-05"
-        iyz="1.9140716904272E-07"
-        izz="4.60418752810541E-05" />
+        value="0.383" />
+      <inertia
+        ixx="0.00166169"
+        ixy="0.00000006"
+        ixz="-0.00000007"
+        iyy="0.00018510"
+        iyz="0.00001026"
+        izz="0.00164321" />
     </inertial>
     <visual>
@@ -349,8 +349,8 @@
         value="0.00699089613564366" />
       <inertia
-        ixx="5.43015540542155E-07"
+        ixx="5.73015540542155E-07"
         ixy="-1.98305403089247E-22"
         ixz="-7.2791893904596E-23"
-        iyy="5.43015540542155E-07"
+        iyy="5.73015540542155E-07"
         iyz="-3.4146026640245E-24"
         izz="1.06738869138926E-06" />
@@ -396,5 +396,5 @@
       upper="2.0944"
       effort="100"
-      velocity="5" />
+      velocity="3" />
   </joint>
 <!-- controller -->
@@ -420,5 +420,5 @@
   <gazebo>
     <plugin name="gazebo_ros_control" filename="libgazebo_ros_control.so">
-        <robotNamespace>/piper_description</robotNamespace>
+        <robotNamespace>/piper</robotNamespace>
         <legacyModeNS>true</legacyModeNS>
     </plugin>

Commit message: [FEAT]更新URDF文件为最新版DH参数

File: src/piper_description/urdf/piper_description.urdf (robot description, URDF)
Before this commit: robot piper, 10 links, 9 joints
Joints:
- joint joint2: origin xyz=0 0 0 rpy=1.5708 -0.10095 -3.1416 -> xyz=0 0 0 rpy=1.5708 -0.1359 -3.1416
- joint joint3: origin xyz=0.28503 0 0 rpy=0 0 -1.759 -> xyz=0.28503 0 0 rpy=0 0 -1.7939

File: src/piper_description/urdf/piper_description.xacro (robot description, xacro)
@@ -153,5 +153,6 @@
     <origin
       xyz="0 0 0"
-      rpy="1.5708 -0.10095 -3.1416" />
+      rpy="1.5708 -0.1359 -3.1416" />
+      <!-- rpy="1.5708 -0.10095-0.03490659 -3.1416" /> -->
     <parent
       link="link1" />
@@ -211,5 +212,6 @@
     <origin
       xyz="0.28503 0 0"
-      rpy="0 0 -1.759" />
+      rpy="0 0 -1.7939" />
+      <!-- rpy="0 0 -1.759-0.03490659" /> -->
     <parent
       link="link2" />

File: src/piper_description/urdf/piper_description_gazebo.xacro (robot description, xacro)
@@ -153,5 +153,6 @@
     <origin
       xyz="0 0 0"
-      rpy="1.5708 -0.10095 -3.1416" />
+      rpy="1.5708 -0.1359 -3.1416" />
+      <!-- rpy="1.5708 -0.10095-0.03490659 -3.1416" /> -->
     <parent
       link="link1" />
@@ -211,5 +212,6 @@
     <origin
       xyz="0.28503 0 0"
-      rpy="0 0 -1.759" />
+      rpy="0 0 -1.7939" />
+      <!-- rpy="0 0 -1.759-0.03490659" /> -->
     <parent
       link="link2" />

File: src/piper_description/urdf/piper_description_old.urdf (robot description, URDF)
Before this commit: robot piper, 7 links, 6 joints
Links:
- added link gripper_base, mass 0.45; collision mesh filename=package://piper_description/meshes/gripper_base.STL; visual mesh filename=package://piper_description/meshes/gripper_base.STL
- added link link7, mass 0.025; collision mesh filename=package://piper_description/meshes/link7.STL; visual mesh filename=package://piper_description/meshes/link7.STL
- added link link8, mass 0.025; collision mesh filename=package://piper_description/meshes/link8.STL; visual mesh filename=package://piper_description/meshes/link8.STL
Joints:
- added joint joint6_to_gripper_base: type fixed, parent link6, child gripper_base, origin xyz=0 0 0 rpy=0 0 0
- added joint joint7: type prismatic, parent gripper_base, child link7, origin xyz=0 0 0.1358 rpy=1.5708 0 0, axis 0 0 1, limit lower=0 upper=0.035 effort=10 velocity=1
- added joint joint8: type prismatic, parent gripper_base, child link8, origin xyz=0 0 0.1358 rpy=1.5708 0 -3.1416, axis 0 0 -1, limit lower=-0.035 upper=0 effort=10 velocity=1
- joint joint2: origin xyz=0 0 0 rpy=1.5708 -0.1359 -3.1416 -> xyz=0 0 0 rpy=1.5708 -0.10095 -3.1416
- joint joint3: origin xyz=0.28503 0 0 rpy=0 0 -1.7939 -> xyz=0.28503 0 0 rpy=0 0 -1.759

File: src/piper_description/urdf/piper_no_gripper_description.xacro (robot description, xacro)
@@ -153,5 +153,6 @@
     <origin
       xyz="0 0 0"
-      rpy="1.5708 -0.10095 -3.1416" />
+      rpy="1.5708 -0.1359 -3.1416" />
+      <!-- rpy="1.5708 -0.10095-0.03490659 -3.1416" /> -->
     <parent
       link="link1" />
@@ -211,5 +212,6 @@
     <origin
       xyz="0.28503 0 0"
-      rpy="0 0 -1.759" />
+      rpy="0 0 -1.7939" />
+      <!-- rpy="0 0 -1.759-0.03490659" /> -->
     <parent
       link="link2" />

File: src/piper_description/urdf/piper_no_gripper_description_gazebo.xacro (robot description, xacro)
@@ -153,5 +153,6 @@
     <origin
       xyz="0 0 0"
-      rpy="1.5708 -0.10095 -3.1416" />
+      rpy="1.5708 -0.1359 -3.1416" />
+      <!-- rpy="1.5708 -0.10095-0.03490659 -3.1416" /> -->
     <parent
       link="link1" />
@@ -211,5 +212,6 @@
     <origin
       xyz="0.28503 0 0"
-      rpy="0 0 -1.759" />
+      rpy="0 0 -1.7939" />
+      <!-- rpy="0 0 -1.759-0.03490659" /> -->
     <parent
       link="link2" />

Commit message: 为urdf文件增加dummy_link;修改moveit默认不编译moveit-1.11包,可以自己apt下载moveit包;增加ros-noetic功能包指示自己当前工作空间是什么版本ros,防止用错误的ros版本编译了错误的工作空间

File: src/piper_description/urdf/piper_description.urdf (robot description, URDF)
Before this commit: robot piper, 10 links, 9 joints
Links:
- added link dummy_link
Joints:
- added joint base_to_dummy: type fixed, parent dummy_link, child base_link, origin xyz=0 0 0 rpy=0 0 0

File: src/piper_description/urdf/piper_no_gripper_description.urdf (robot description, URDF)
Before this commit: robot piper, 7 links, 6 joints
Links:
- added link dummy_link
Joints:
- added joint base_to_dummy: type fixed, parent dummy_link, child base_link, origin xyz=0 0 0 rpy=0 0 0

Commit message: 修改urdf中link6的质量为0.007kg

File: src/piper_description/urdf/piper_description.urdf (robot description, URDF)
Before this commit: robot piper, 11 links, 10 joints
Links:
- link link6: mass 0.00699089613564366 -> 0.007

File: src/piper_description/urdf/piper_description.xacro (robot description, xacro)
@@ -349,5 +349,5 @@
         rpy="0 0 0" />
       <mass
-        value="0.00699089613564366" />
+        value="0.007" />
       <inertia
         ixx="5.73015540542155E-07"

File: src/piper_description/urdf/piper_description_gazebo.xacro (robot description, xacro)
@@ -349,5 +349,5 @@
         rpy="0 0 0" />
       <mass
-        value="0.00699089613564366" />
+        value="0.007" />
       <inertia
         ixx="5.73015540542155E-07"

File: src/piper_description/urdf/piper_description_old.urdf (robot description, URDF)
Before this commit: robot piper, 10 links, 9 joints
Links:
- link link6: mass 0.00699089613564366 -> 0.007

File: src/piper_description/urdf/piper_no_gripper_description.urdf (robot description, URDF)
Before this commit: robot piper, 8 links, 7 joints
Links:
- link link6: mass 0.00699089613564366 -> 0.007

File: src/piper_description/urdf/piper_no_gripper_description.xacro (robot description, xacro)
@@ -349,5 +349,5 @@
         rpy="0 0 0" />
       <mass
-        value="0.00699089613564366" />
+        value="0.007" />
       <inertia
         ixx="5.73015540542155E-07"

File: src/piper_description/urdf/piper_no_gripper_description_gazebo.xacro (robot description, xacro)
@@ -349,5 +349,5 @@
         rpy="0 0 0" />
       <mass
-        value="0.00699089613564366" />
+        value="0.007" />
       <inertia
         ixx="5.73015540542155E-07"

File: src/piper_description/urdf/piper_no_gripper_description_old.urdf (robot description, URDF)
Before this commit: robot piper, 7 links, 6 joints
Links:
- link link6: mass 0.00699089613564366 -> 0.007
