Commit message: modify the position of D435camera

File: src/piper_description/urdf/piper_no_gripper_description_realsense_gazebo.xacro (robot description, xacro)
@@ -410,5 +410,5 @@
     </inertial>
     <visual>
-      <origin xyz="0 0 0.01" rpy="1.57 0 1.57" />
+      <origin xyz="0.014 0 0.00" rpy="1.57 0 1.57" />
       <geometry>
         <mesh filename="package://piper_description/meshes/d435.dae" />
