Commit message: Calibrate the depth camera's viewpoint to match that of the image_raw

File: src/piper_description/urdf/piper_no_gripper_description_realsense_gazebo.urdf (robot description, URDF)
Before this commit: robot gazebo, 9 links, 8 joints
Links:
- added link camera_color_optical_frame
- added link camera_depth_optical_frame
- added link camera_infra1_optical_frame
- added link camera_infra2_optical_frame
Joints:
- added joint camera_color_optical_joint: type fixed, parent d435_link, child camera_color_optical_frame, origin xyz=0 0 0 rpy=1.5708 0 1.5708
- added joint camera_depth_optical_joint: type fixed, parent d435_link, child camera_depth_optical_frame, origin xyz=0 0 0 rpy=1.5708 0 0
- added joint camera_infra1_optical_joint: type fixed, parent d435_link, child camera_infra1_optical_frame, origin xyz=0 0 0 rpy=1.5708 0 1.5708
- added joint camera_infra2_optical_joint: type fixed, parent d435_link, child camera_infra2_optical_frame, origin xyz=0 0 0 rpy=1.5708 0 1.5708
- joint d435_joint: origin xyz=0 0 0.01 rpy=0 -1.57 0 -> xyz=0 0 0.01 rpy=0 -1.57 3.14

File: src/piper_description/urdf/piper_no_gripper_description_realsense_gazebo.xacro (robot description, xacro)
@@ -428,5 +428,5 @@
   </joint>
   <!-- D435光学坐标系 -->
-  <!-- <link name="camera_color_optical_frame">
+  <link name="camera_color_optical_frame">
     <visual>
       <origin xyz="0 0 0" rpy="1.5708 0 1.5708" />
@@ -437,13 +437,13 @@
     <parent link="d435_link" />
     <child link="camera_color_optical_frame" />
-  </joint> -->
+  </joint>
   <!-- 其他D435光学坐标系 -->
-  <!-- <link name="camera_depth_optical_frame">
-    <visual>
-      <origin xyz="0 0 0" rpy="0 0 1.5708" />
+  <link name="camera_depth_optical_frame">
+    <visual>
+      <origin xyz="0 0 0" rpy="0 0 3.14" />
     </visual>
   </link>
   <joint name="camera_depth_optical_joint" type="fixed">
-    <origin xyz="0 0 0" rpy="1.5708 0 1.5708" />
+    <origin xyz="0 0 0" rpy="1.5708 0 0" />
     <parent link="d435_link" />
     <child link="camera_depth_optical_frame" />
@@ -468,5 +468,5 @@
     <parent link="d435_link" />
     <child link="camera_infra2_optical_frame" />
-  </joint> -->
+  </joint>
   <!-- 实例化D435宏 -->
   <xacro:gazebo_d435
